File: NE555-Arduino_interrupt_source/NE555_Arduino_interrupt_source.sch (EAGLE design)
At the start: 9 parts, among them IC1 NE555

Commit message: Faster output
Parts:
- C1: value 100uF -> 0,01uF
Other:
- note added: "Output about 250Hz-11kHz"
Changed lines of the file:
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@@
 <part name="VR1" library="pot" library_urn="urn:adsk.eagle:library:331" deviceset="3RP/1610N" device="" package3d_urn="urn:adsk.eagle:package:22726/1" value="250kOhm"/>
 <part name="C2" library="capacitor-wima" library_urn="urn:adsk.eagle:library:116" deviceset="C" device="2,5-3" package3d_urn="urn:adsk.eagle:package:5436/1" value="0,01uF"/>
-<part name="C1" library="capacitor-wima" library_urn="urn:adsk.eagle:library:116" deviceset="C" device="2,5-3" package3d_urn="urn:adsk.eagle:package:5436/1" value="100uF"/>
+<part name="C1" library="capacitor-wima" library_urn="urn:adsk.eagle:library:116" deviceset="C" device="2,5-3" package3d_urn="urn:adsk.eagle:package:5436/1" value="0,01uF"/>
 <part name="GND1" library="supply1" library_urn="urn:adsk.eagle:library:371" deviceset="GND" device=""/>
 <part name="R2" library="rcl" library_urn="urn:adsk.eagle:library:334" deviceset="R-EU_" device="0204/2V" package3d_urn="urn:adsk.eagle:package:23495/1" value="4,7kOhm"/>
@@
 <sheet>
 <plain>
+<text x="91.44" y="71.12" size="1.778" layer="91">Output about 250Hz-11kHz</text>
 </plain>
 <instances>
